Commit message: fix cs

File: urdf/MontyURDF.urdf (robot description, URDF)
Before this commit: robot MontyURDF, 3 links, 2 joints
Links:
- link base_link: mass 1.84635819081325 -> 1.88328535462952; geometry collision mesh filename=package://montyurdf/meshes/base_link.STL; visual mesh filename=package://montyurdf/meshes/base_link.STL
- link left_wheel_link: geometry collision mesh filename=package://montyurdf/meshes/left_wheel_link.STL; visual mesh filename=package://montyurdf/meshes/left_wheel_link.STL
- link right_wheel_link: geometry collision mesh filename=package://montyurdf/meshes/right_wheel_link.STL; visual mesh filename=package://montyurdf/meshes/right_wheel_link.STL
Joints:
- joint leftWheelJoint: axis 1 0 0 -> 0 1 0; limit (none) -> effort=1 velocity=1; origin xyz=0.095 0.015 -0.066858 rpy=0 0 0 -> xyz=-0.066858 0.095 0.015 rpy=0 0 0
- joint rightWheelJoint: axis 1 0 0 -> 0 1 0; limit (none) -> effort=1 velocity=1; origin xyz=-0.095 0.015 -0.066858 rpy=0 0 0 -> xyz=-0.066858 -0.095 0.015 rpy=0 0 0
